Commit message: Fix gimbal-camera TF: use camera_link as optical frame and correct rotation

File: venom_robot_description/urdf/rm_gimbal.urdf.xacro (robot description, xacro)
@@ -2,5 +2,5 @@
 <robot name="rm_gimbal"
   xmlns:xacro="http://ros.org/wiki/xacro">
-  <xacro:arg name="xyz" default="0.10 0 0.05" />
+  <xacro:arg name="xyz" default="0.04 0.11 0.02" />
   <xacro:arg name="rpy" default="0 0 0" />
   <link name="odom" />
@@ -11,15 +11,3 @@
   </joint>
   <link name="camera_link" />
-  <joint name="camera_joint" type="fixed">
-    <origin xyz="$(arg xyz)" rpy="$(arg rpy)" />
-    <parent link="gimbal_link" />
-    <child link="camera_link" />
-    <axis xyz="0 0 0" />
-  </joint>
-  <link name="camera_optical_frame" />
-  <joint name="camera_optical_joint" type="fixed">
-    <origin xyz="0 0 0" rpy="${-pi/2} 0 ${-pi/2}" />
-    <parent link="camera_link" />
-    <child link="camera_optical_frame" />
-  </joint>
 </robot>
